File: PIC_QuickDevBoard.kicad_sch (KiCad schematic)
At the start: 36 parts, among them J1 Conn_01x08_Pin, J10 VCC Lines, J2 Conn_01x08_Pin, J3 Conn_01x08_Pin, J4 PowerSource, J5 PICKitConnector, J6 USB_B_Micro, J7 PGEC_LINES, J8 PGED_LINES, J9 MCLR_LINES, SW1 SW_Push, U1 PIC24F, U2 PIC16F84, U3 LDA33A, U4 PIC16F1459-IP, Y1 Crystal

Commit message: Rev2.3 - led on RB4 and Demo for all three suported PICs
Connections:
- net RA1: no longer R4.1
- net RB4: now also R4.1
Changed lines of the file:
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@@
 	(title_block
 		(title "PIC24 & PIC16F84 Programmer & Dev Board")
-		(date "2024-05-17")
+		(date "2024-05-19")
 		(rev "2.3")
 		(company "RCC 2024")
@@
 		)
 	)
-	(global_label "RC0"
-		(shape bidirectional)
-		(at 396.24 102.87 180)
-		(fields_autoplaced yes)
-		(effects
-			(font
-				(size 1.27 1.27)
-			)
-			(justify right)
-		)
-		(property "Intersheetrefs" "${INTERSHEET_REFS}"
-			(at 388.394 102.87 0)
-			(effects
-				(font
-					(size 1.27 1.27)
-				)
-				(justify right)
-				(hide yes)
-			)
-		)
-	)
-	(global_label "RB1"
-		(shape bidirectional)
-		(at 119.4867 105.4238 0)
-		(fields_autoplaced yes)
-		(effects
-			(font
-				(size 1.27 1.27)
-			)
-			(justify left)
-		)
-		(property "Intersheetrefs" "${INTERSHEET_REFS}"
-			(at 127.3327 105.4238 0)
-			(effects
-				(font
-					(size 1.27 1.27)
-				)
-				(justify left)
-				(hide yes)
-			)
-		)
-	)
-	(global_label "RC1"
-		(shape bidirectional)
-		(at 374.65 105.41 0)
-		(fields_autoplaced yes)
-		(effects
-			(font
-				(size 1.27 1.27)
-			)
-			(justify left)
-		)
-		(property "Intersheetrefs" "${INTERSHEET_REFS}"
-			(at 382.496 105.41 0)
-			(effects
-				(font
-					(size 1.27 1.27)
-				)
-				(justify left)
-				(hide yes)
-			)
-		)
-	)
-	(global_label "RA1"
+	(global_label "RB4"
 		(shape input)
 		(at 233.432 211.9811 0)
@@
 		)
 		(property "Intersheetrefs" "${INTERSHEET_REFS}"
-			(at 239.9853 211.9811 0)
-			(effects
-				(font
+			(at 240.1667 211.9811 0)
+			(effects
+				(font
+					(size 1.27 1.27)
+				)
+				(justify left)
+				(hide yes)
+			)
+		)
+	)
+	(global_label "RC0"
+		(shape bidirectional)
+		(at 396.24 102.87 180)
+		(fields_autoplaced yes)
+		(effects
+			(font
+				(size 1.27 1.27)
+			)
+			(justify right)
+		)
+		(property "Intersheetrefs" "${INTERSHEET_REFS}"
+			(at 388.394 102.87 0)
+			(effects
+				(font
+					(size 1.27 1.27)
+				)
+				(justify right)
+				(hide yes)
+			)
+		)
+	)
+	(global_label "RB1"
+		(shape bidirectional)
+		(at 119.4867 105.4238 0)
+		(fields_autoplaced yes)
+		(effects
+			(font
+				(size 1.27 1.27)
+			)
+			(justify left)
+		)
+		(property "Intersheetrefs" "${INTERSHEET_REFS}"
+			(at 127.3327 105.4238 0)
+			(effects
+				(font
+					(size 1.27 1.27)
+				)
+				(justify left)
+				(hide yes)
+			)
+		)
+	)
+	(global_label "RC1"
+		(shape bidirectional)
+		(at 374.65 105.41 0)
+		(fields_autoplaced yes)
+		(effects
+			(font
+				(size 1.27 1.27)
+			)
+			(justify left)
+		)
+		(property "Intersheetrefs" "${INTERSHEET_REFS}"
+			(at 382.496 105.41 0)
+			(effects
+				(font
